Commit message: Avec la camera 2

File: robot_tennis_description/urdf/robot.urdf.xacro (robot description, xacro)
@@ -189,43 +189,6 @@
     <xacro:fixed_joint elem1="${name}_4" elem2="${name}_aruco_11" />
   </xacro:macro>
-  <xacro:macro name="wheel" params="name ep r m">
-    <link name="wheel_${name}">
-    <visual>
-      <geometry>
-        <cylinder length="${ep}" radius="${r}"/>
-      </geometry>
-    </visual>
-    <collision>
-      <geometry>
-        <cylinder length="${ep}" radius="${r}"/>
-      </geometry>
-    </collision>
-    <inertial>
-      <mass value="${m}"/>
-      <xacro:cylinder_inertia m="${m}" r="${r}" h="${ep}"/>
-    </inertial>
-    </link>
-    <gazebo reference="wheel_${name}">
-      <mu1>1.2</mu1>
-      <mu2>1.2</mu2>
-      <kp>500000.0</kp>
-      <kd>10.0</kd>
-      <minDepth>0.001</minDepth>
-      <maxVel>0.1</maxVel>
-      <material>Gazebo/FlatBlack</material>
-    </gazebo>
-  </xacro:macro>
-  <link name="root_link"/>
-  <joint name="root_to_bloc_1" type="fixed">
-    <parent link="root_link"/>
-    <child link="center_1"/>
-  </joint>
-  <xacro:bloc4 name="center" x="0.0" y="0.0" z="0.175" l1="0.8" l2="0.4" h="0.4" ep="0.05" m="10" />
-  <xacro:bloc5 name="catcher" x="-0.375" y="0.0" z="0.175" l="0.275" h="0.3" ep="0.01" m="3" />
-  <xacro:wheel name="left_front" r="0.20" ep="0.15" m="3"/>
-  <xacro:wheel name="left_back" r="0.20" ep="0.15" m="3"/>
-  <xacro:wheel name="right_front" r="0.20" ep="0.15" m="3"/>
-  <xacro:wheel name="right_back" r="0.20" ep="0.15" m="3"/>
-  <link name="camera_link">
+  <xacro:macro name="camera_xacro" params="name">
+  <link name="${name}">
     <collision>
       <origin xyz="0 0 0" rpy="0 0 0"/>
@@ -247,5 +210,46 @@
     </inertial>
   </link>
-  <gazebo reference="camera_link">
+  </xacro:macro>
+  <xacro:macro name="wheel" params="name ep r m">
+    <link name="wheel_${name}">
+    <visual>
+      <geometry>
+        <cylinder length="${ep}" radius="${r}"/>
+      </geometry>
+    </visual>
+    <collision>
+      <geometry>
+        <cylinder length="${ep}" radius="${r}"/>
+      </geometry>
+    </collision>
+    <inertial>
+      <mass value="${m}"/>
+      <xacro:cylinder_inertia m="${m}" r="${r}" h="${ep}"/>
+    </inertial>
+    </link>
+    <gazebo reference="wheel_${name}">
+      <mu1>1.2</mu1>
+      <mu2>1.2</mu2>
+      <kp>500000.0</kp>
+      <kd>10.0</kd>
+      <minDepth>0.001</minDepth>
+      <maxVel>0.1</maxVel>
+      <material>Gazebo/FlatBlack</material>
+    </gazebo>
+  </xacro:macro>
+  <link name="root_link"/>
+  <joint name="root_to_bloc_1" type="fixed">
+    <parent link="root_link"/>
+    <child link="center_1"/>
+  </joint>
+  <xacro:bloc4 name="center" x="0.0" y="0.0" z="0.175" l1="0.8" l2="0.4" h="0.4" ep="0.05" m="10" />
+  <xacro:bloc5 name="catcher" x="-0.375" y="0.0" z="0.175" l="0.275" h="0.3" ep="0.01" m="3" />
+  <xacro:wheel name="left_front" r="0.20" ep="0.15" m="3"/>
+  <xacro:wheel name="left_back" r="0.20" ep="0.15" m="3"/>
+  <xacro:wheel name="right_front" r="0.20" ep="0.15" m="3"/>
+  <xacro:wheel name="right_back" r="0.20" ep="0.15" m="3"/>
+  <xacro:camera_xacro name="camera1_link" />
+  <xacro:camera_xacro name="camera2_link" />
+  <gazebo reference="camera1_link">
     <sensor name="camera1" type="camera">
         <always_on>1</always_on>
@@ -269,8 +273,36 @@
     </sensor>
   </gazebo>
-  <joint name="catcher_to_cam0" type="fixed">
+  <gazebo reference="camera2_link">
+    <sensor name="camera2" type="camera">
+        <always_on>1</always_on>
+        <update_rate>10</update_rate>
+        <visualize>true</visualize>
+        <camera name="camera2">
+            <horizontal_fov>1</horizontal_fov>
+            <image>
+                <width>800</width>
+                <height>800</height>
+            </image>
+            <clip>
+                <near>0.02</near>
+                <far>300</far>
+            </clip>
+        </camera>
+        <plugin name="camera2_controller" filename="libgazebo_ros_camera.so">
+            <camera_name>camera2</camera_name>
+            <hack_baseline>0.07</hack_baseline>
+        </plugin>
+    </sensor>
+  </gazebo>
+  <joint name="catcher_to_cam1" type="fixed">
     <parent link="catcher_5"/>
-    <child link="camera_link"/>
+    <child link="camera1_link"/>
     <origin rpy="0 1.57075 0" xyz="-0.375 0 0.475"/>
+    <axis xyz= "0 0 1"/>
+  </joint>
+  <joint name="catcher_to_cam2" type="fixed">
+    <parent link="catcher_5"/>
+    <child link="camera2_link"/>
+    <origin rpy="0 2 0" xyz="-0.525 0 0.475"/>
     <axis xyz= "0 0 1"/>
   </joint>

Commit message: tmp

File: robot_tennis_description/urdf/robot.urdf.xacro (robot description, xacro)
@@ -189,5 +189,5 @@
     <xacro:fixed_joint elem1="${name}_4" elem2="${name}_aruco_11" />
   </xacro:macro>
-  <xacro:macro name="camera_xacro" params="name">
+  <xacro:macro name="sensor_xacro" params="name">
   <link name="${name}">
     <collision>
@@ -249,6 +249,7 @@
   <xacro:wheel name="right_front" r="0.20" ep="0.15" m="3"/>
   <xacro:wheel name="right_back" r="0.20" ep="0.15" m="3"/>
-  <xacro:camera_xacro name="camera1_link" />
-  <xacro:camera_xacro name="camera2_link" />
+  <xacro:sensor_xacro name="camera1_link" />
+  <xacro:sensor_xacro name="camera2_link" />
+  <xacro:sensor_xacro name="imu_link" />
   <gazebo reference="camera1_link">
     <sensor name="camera1" type="camera">
@@ -295,8 +296,29 @@
     </sensor>
   </gazebo>
+  <gazebo reference="imu_link">
+    <sensor name="imu0" type="imu">
+    <always_on>true</always_on>
+    <!-- Publish at 30 hz -->
+    <update_rate>30</update_rate>
+    <plugin name="imu0_plugin" filename="libgazebo_ros_imu_sensor.so">
+      <ros>
+        <!-- Will publish to /imu/data -->
+        <namespace>/imu</namespace>
+        <argument>~/out:=data</argument>
+      </ros>
+      <!-- frame_name ommited, will be "my_link" -->
+    </plugin>
+  </sensor>
+  </gazebo>
   <joint name="catcher_to_cam1" type="fixed">
     <parent link="catcher_5"/>
     <child link="camera1_link"/>
     <origin rpy="0 1.57075 0" xyz="-0.375 0 0.475"/>
+    <axis xyz= "0 0 1"/>
+  </joint>
+  <joint name="catcher_to_imu" type="fixed">
+    <parent link="catcher_5"/>
+    <child link="imu_link"/>
+    <origin rpy="0 0 0" xyz="0 0 0.25"/>
     <axis xyz= "0 0 1"/>
   </joint>

Commit message: GPS dispo sous gazebo

File: robot_tennis_description/urdf/robot.urdf.xacro (robot description, xacro)
@@ -252,4 +252,5 @@
   <xacro:sensor_xacro name="camera2_link" />
   <xacro:sensor_xacro name="imu_link" />
+  <xacro:sensor_xacro name="gps_link" />
   <gazebo reference="camera1_link">
     <sensor name="camera1" type="camera">
@@ -320,4 +321,18 @@
   </sensor>
   </gazebo>-->
+<gazebo reference="gps_link">
+    <sensor name="gps_sensor" type="gps">
+	<always_on>true</always_on>
+	<update_rate>10</update_rate>
+	<plugin name="gps_controller" filename="libgazebo_ros_gps_sensor.so">
+	    <ros>
+		<!-- <namespace>/br</namespace> -->
+		<remapping>gps_controller/out:=gps</remapping>
+	    </ros>
+	    <frame_name>gps_link</frame_name>
+	</plugin>
+    </sensor>
+    <material>Gazebo/Grey</material>
+</gazebo>
   <joint name="catcher_to_cam1" type="fixed">
     <parent link="catcher_5"/>
@@ -367,4 +382,10 @@
     <axis xyz="0 0 1"/>
     <limit effort="10" lower="-0.10" upper="0.0" velocity="0.5"/>
+  </joint>
+  <joint name="catcher_to_gps" type="fixed">
+    <parent link="catcher_5"/>
+    <child link="gps_link"/>
+    <origin rpy="0 0 0" xyz="0 0 0.25"/>
+    <axis xyz= "0 0 1"/>
   </joint>
   <gazebo>
